Commit message: fix dropped gripper joints + perception startup diagnostics
urdf: give tool0 a small inertial and preserve tool0_joint/camera_joint.
Gazebo Classic lumps fixed joints into the parent link; with a massless
tool0 the two finger joints hanging off it were removed from the SDF, so
gazebo_ros2_control skipped finger_left/finger_right and
gripper_controller failed to activate ('prepare command mode switch was
rejected').

perception: readiness no longer depends on a single message field. Use
joint velocities, fall back to position deltas, tolerate a missing
/ag_execution/ready latch after a 20 s grace window, and log a
'not calibrated yet: <reason>' line every 3 s. env: wait up to 120 s for
the first calibrated observation instead of 40 s.

File: src/ag_description/urdf/ag_arm.urdf (robot description, URDF)
Before this commit: robot ag_arm, 11 links, 10 joints
Links:
- link tool0: mass None -> 0.02
