Commit message: fix grasp execution: threading, fingertip depth, gripper geometry
The gripper exists (both finger joints are in /joint_states) but the demo
could never grasp because of three real defects:

1. Every trajectory was reported as 'arm controller did not answer the goal
   request': the node pumped rclpy.spin_once from inside its own service
   callback, which stops delivering action results. Switch to a
   MultiThreadedExecutor(3), give the four services their own mutually
   exclusive callback group, move the startup motion into startup() and let
   blocking waits only sleep while executor threads deliver callbacks.
2. grasp_plan used a constant grasp_offset, so the fingertips stopped 5 mm
   below the object top for every object size - a top-edge pinch that always
   slips. Place the fingertips at half the object height instead:
   tool_z = max(0.01, 0.5*z_top) + finger_length (0.07), never closer than
   1 cm to the table.
3. Fingers were 1.6x2 cm and washed out; widen to 2x2.6x6 cm (4 cm gap, 4 mm
   closed), give them Gazebo/DarkGrey so they are visible, cap object sizes
   at 4 cm so they fit between the jaws, and lower the bin drop pose to
   z=0.29 (IK error 13mm -> 4.5mm).

Tests: 22 passing (adds fingertip-depth coverage).

File: src/ag_description/urdf/ag_arm.urdf (robot description, URDF)
Before this commit: robot ag_arm, 11 links, 10 joints
Links:
- link finger_left_link: geometry collision box size=0.02 0.026 0.06; visual box size=0.02 0.026 0.06
- link finger_right_link: geometry collision box size=0.02 0.026 0.06; visual box size=0.02 0.026 0.06
Joints:
- joint finger_left: origin xyz=-0.028 0 -0.01 rpy=0 0 0 -> xyz=-0.030 0 -0.01 rpy=0 0 0
- joint finger_right: origin xyz=0.028 0 -0.01 rpy=0 0 0 -> xyz=0.030 0 -0.01 rpy=0 0 0

Commit message: widen gripper clearance and make grasp failures diagnosable
Objects are up to 3.4 cm wide but the jaws only opened 4.0 cm, leaving
3 mm per side: the descending fingers knock the object away and then close
on air (hold check fails, reward -0.30). Open the jaws to 5.2 cm (closed
gap 1.6 cm) and judge a grasp by the real gap: closed gap + 4 mm.

Also stop hiding motion: the push reward averaged |dh| over all 48x48
cells, so moving one object changed the mean by ~0.0005 and every push
looked like it did nothing. Average over occupied cells only.

New diagnostics to settle the remaining question with data:
- execution logs 'grasp cell (u,v) -> (x, y), z_top, descend, held, width'
- perception logs the three tallest heightmap cells in world coordinates
- env logs gripper width and push delta

Hold detection moved into primitives (gripper_width / is_holding) with
unit tests; 23 passing. FK cross-checked against yourdfpy (max element
error 2e-12 over random configurations).

File: src/ag_description/urdf/ag_arm.urdf (robot description, URDF)
Before this commit: robot ag_arm, 11 links, 10 joints
Joints:
- joint finger_left: origin xyz=-0.030 0 -0.01 rpy=0 0 0 -> xyz=-0.036 0 -0.01 rpy=0 0 0
- joint finger_right: origin xyz=0.030 0 -0.01 rpy=0 0 0 -> xyz=0.036 0 -0.01 rpy=0 0 0

Commit message: grasp objects by their blob centre, gently, and verify them in gazebo
Latest run proves the arm side is exact: 'tool pose: commanded
(0.424, -0.089, 0.076) actual (0.424, -0.089, 0.076) error=0.0 mm' while
'width_at_hold=0.0160' means the jaws closed completely - so nothing was
between them even though the height map placed the object ~1 cm away.
The objects are being shoved aside by the approach/closing, not missed by
the controller.

- env: snap the grasp cell to the centroid of the local occupied blob
  (actions.blob_centre) instead of the tallest cell, which is usually the
  rim of the object.
- execution: descend 0.55 -> 1.1 s and close 0.7 -> 1.4 s so contacts can
  settle instead of batting the object away.
- urdf: finger pads 2.6 -> 3.2 cm deep and mu 1.0 -> 1.5 for more contact.
- world: load gazebo_ros_state; on a failed grasp the execution node logs
  every ag_obj_* world position and its distance to the grasp point, so
  the next run shows whether the object was knocked away or never there.
- tests: 24 passing (adds blob-centre coverage).

File: src/ag_description/urdf/ag_arm.urdf (robot description, URDF)
Before this commit: robot ag_arm, 11 links, 10 joints
Links:
- link finger_left_link: geometry collision box size=0.02 0.032 0.06; visual box size=0.02 0.032 0.06
- link finger_right_link: geometry collision box size=0.02 0.032 0.06; visual box size=0.02 0.032 0.06

Commit message: widen jaw travel and log grasp-point snapping
Rotated log from the lab: 'tool pose ... error=0.0 mm' for nearly every
move, 'width_at_hold=0.0160' (jaws fully closed) and pushes that move the
clutter by up to 21 mm. So the fingers exist and work, the arm is on
target, and the object is being shoved out during the top-down grasp.

That run also shows no 'object ag_obj_*' lines and grasp cells that keep
alternating between (20,33)/(21,33): it was built from the previous commit,
so the centroid snapping and slower motions had not been tested yet. Make
the approach even more forgiving:

- jaws open 5.2 -> 5.6 cm with 2.6 cm stroke (closed 0.4 cm): 11 mm
  clearance per side around a 3.4 cm object.
- demo logs 'grasp snapped from (u,v) to (u,v)' so the centroid step is
  visible in the log.
- docs updated; tests 24 passing.

File: src/ag_description/urdf/ag_arm.urdf (robot description, URDF)
Before this commit: robot ag_arm, 11 links, 10 joints
Joints:
- joint finger_left: limit lower=0 upper=0.018 effort=25 velocity=0.03 -> lower=0 upper=0.026 effort=25 velocity=0.04; origin xyz=-0.036 0 -0.01 rpy=0 0 0 -> xyz=-0.038 0 -0.01 rpy=0 0 0
- joint finger_right: limit lower=0 upper=0.018 effort=25 velocity=0.03 -> lower=0 upper=0.026 effort=25 velocity=0.04; origin xyz=0.036 0 -0.01 rpy=0 0 0 -> xyz=0.038 0 -0.01 rpy=0 0 0

Commit message: anchor the robot base and widen the jaws to stop knocking objects away
This run reached the object but two structural problems appeared:

1. The whole arm toppled off the table once the fingers touched something:
   the base was a free-floating 2 kg body and the arm reaches ~1 m. Widen
   the foot to 24 cm, raise its mass to 20 kg and mark base_link
   kinematic so the base is anchored to the world while the joints still
   move.
2. The object was knocked 7-11 cm away during the descent (jaws still
   closed to the 0.4 cm gap afterwards, i.e. nothing was ever between
   them). Open the jaws to 7.0 cm (1.8 cm clearance per side for a 3.4 cm
   object), stroke 3.4 cm, closed gap 0.2 cm, and slow the descent to
   1.8 s.

Tests: 27 passing.

File: src/ag_description/urdf/ag_arm.urdf (robot description, URDF)
Before this commit: robot ag_arm, 11 links, 10 joints
Links:
- link base_link: mass 2.0 -> 20.0; geometry collision box size=0.24 0.24 0.12; visual box size=0.24 0.24 0.12
Joints:
- joint finger_left: limit lower=0 upper=0.026 effort=25 velocity=0.04 -> lower=0 upper=0.034 effort=25 velocity=0.05; origin xyz=-0.038 0 -0.01 rpy=0 0 0 -> xyz=-0.045 0 -0.01 rpy=0 0 0
- joint finger_right: limit lower=0 upper=0.026 effort=25 velocity=0.04 -> lower=0 upper=0.034 effort=25 velocity=0.05; origin xyz=0.038 0 -0.01 rpy=0 0 0 -> xyz=0.045 0 -0.01 rpy=0 0 0

Commit message: make the jaws visible and judge contact from the achieved joint position
Log analysis: the base anchor works (the arm stays up) and the descent no
longer flings the object (delta 2.6 mm), but contact detection still fired
falsely (negative movement means the jaws were still opening from the
previous action), and a stalled joint (-1.39 rad) came from the fingertips
catching the table.

- _grasp_close: open the jaws first (0.8 s), then step in; contact is now
  achieved finger position < 0.6 * commanded.
- grasp_plan: descend only to 1.5 cm above the table.
- fingers: orange, 7 cm pads (tips 8 cm below tool0), slightly wider.
- tests 27 passing.

File: src/ag_description/urdf/ag_arm.urdf (robot description, URDF)
Before this commit: robot ag_arm, 11 links, 10 joints
Links:
- link finger_left_link: geometry collision box size=0.02 0.034 0.07; visual box size=0.02 0.034 0.07
- link finger_right_link: geometry collision box size=0.02 0.034 0.07; visual box size=0.02 0.034 0.07

Commit message: rebuild the gripper as a real parallel jaw and fix slow-loop contact detection
The old gripper was two floating pads with no palm, which reads as random
orange cubes in Gazebo and gives the fingers nothing to mount on. New
model: gripper_base palm (11x6x2 cm, dark grey) fixed to tool0 (preserved
against fixed-joint lumping) with two orange fingers (1.6x3.2x7.5 cm) on
prismatic joints; open gap 6.4 cm, closed 0.4 cm, fingertips 10.5 cm below
tool0.

Log analysis of type (9): almost every grasp closed to the 0.4 cm gap
with height-map delta ~0, i.e. the fingers closed on air, and the two
jaw-contact detections fired at q=0.0043 with achieved 0.0001-0.0020 -
the gazebo position loop is a slow first-order response, so 0.3 s steps
never finish. The close routine now settles the open gripper first, then
closes in 4 steps of 0.9 s and treats less than 25% of the expected width
change as contact. Arm trajectory durations are lengthened again (2.0-2.8 s)
because the same slow loop caused 0.1-0.26 rad tracking aborts.

Tests: 27 passing.

File: src/ag_description/urdf/ag_arm.urdf (robot description, URDF)
Before this commit: robot ag_arm, 11 links, 10 joints
Links:
- added link gripper_base, mass 0.3; collision box size=0.11 0.06 0.02; visual box size=0.11 0.06 0.02
- link finger_left_link: mass 0.05 -> 0.06; geometry collision box size=0.016 0.032 0.075; visual box size=0.016 0.032 0.075
- link finger_right_link: mass 0.05 -> 0.06; geometry collision box size=0.016 0.032 0.075; visual box size=0.016 0.032 0.075
Joints:
- added joint gripper_base_joint: type fixed, parent tool0, child gripper_base, origin xyz=0 0 0 rpy=0 0 0
- joint finger_left: limit lower=0 upper=0.034 effort=25 velocity=0.05 -> lower=0 upper=0.030 effort=30 velocity=0.10; origin xyz=-0.045 0 -0.01 rpy=0 0 0 -> xyz=-0.040 0 -0.030 rpy=0 0 0; parent tool0 -> gripper_base
- joint finger_right: limit lower=0 upper=0.034 effort=25 velocity=0.05 -> lower=0 upper=0.030 effort=30 velocity=0.10; origin xyz=0.045 0 -0.01 rpy=0 0 0 -> xyz=0.040 0 -0.030 rpy=0 0 0; parent tool0 -> gripper_base

Commit message: limit joint travel and keep one IK branch
Log: the grasp itself now works (jaw contact, width 0.032, held=True) but
the transit to the bin aborted with errors on every joint (0.1 to 3.0 rad).
Numerically, home -> approach moved joint5 by 2.93 rad and consecutive
waypoints jumped 0.8 rad because IK flipped between elbow-up and
elbow-down branches.

- URDF: joint2 +-2.2 (was +-2.8), joint3 -2.2..1.6 (was +-2.8),
  joint4/joint5 +-2.6 (was +-3.14). The home pose no longer sits at
  joint5 = +-pi.
- kinematics.ik: posture regularisation towards the seed (0.03) keeps
  consecutive solutions in the same branch; ik_retry tries 12 random seeds.
- execution: max_joint_speed=0.6 rad/s; trajectories are stretched when a
  large configuration change is requested.
- world_manager: clutter spawns only in the verified-reachable box
  x 0.40..0.62, y +-0.12.
- tests: 28 passing (adds a continuity test for approach/descend/lift and a
  workspace grid over the spawn box).

File: src/ag_description/urdf/ag_arm.urdf (robot description, URDF)
Before this commit: robot ag_arm, 12 links, 11 joints
Joints:
- joint joint2: limit lower=-2.8 upper=2.8 effort=80 velocity=2.0 -> lower=-2.2 upper=2.2 effort=80 velocity=2.0
- joint joint3: limit lower=-2.8 upper=2.8 effort=60 velocity=2.5 -> lower=-2.2 upper=1.6 effort=60 velocity=2.5
- joint joint4: limit lower=-3.1416 upper=3.1416 effort=40 velocity=3.0 -> lower=-2.6 upper=2.6 effort=40 velocity=3.0
- joint joint5: limit lower=-3.1416 upper=3.1416 effort=30 velocity=3.0 -> lower=-2.6 upper=2.6 effort=30 velocity=3.0

Commit message: point the wrist camera the same way as the fingers and move the home pose over the table
Two geometric causes made the intermediate joints sweep absurdly:

1. The old home camera pose (0.68,0,0.62) has an IK solution with joint1 = pi,
   so the whole arm started facing backwards and had to swing 180 degrees
   before every grasp (the 3.1 rad stretches, sometimes ending 1 m off).
2. The camera looked along +tool z while the fingers hang along -tool z, so
   looking at the table put the gripper upside down and every grasp needed a
   180 degree wrist turn.

- camera_joint rpy (0,-pi/2,0) -> (0,+pi/2,0): camera now looks along -tool z,
  same direction as the fingers; perception v_sign becomes +1 (u stays -1).
- home camera pose (0.50,0,0.70) looking at (0.50,0,0.02): IK gives
  joint1 = 0, and home -> approach maximum joint change drops from 3.10 rad
  to 1.01 rad (descend/lift 0.40 rad).
- tests updated for the new camera axis; 28 passing.

File: src/ag_description/urdf/ag_arm.urdf (robot description, URDF)
Before this commit: robot ag_arm, 12 links, 11 joints
Joints:
- joint camera_joint: origin xyz=0.06 0 0.04 rpy=0 -1.5708 0 -> xyz=0.06 0 0.04 rpy=0 1.5708 0
